File: thinkmods-re.kicad_sch (KiCad schematic)
At the start: 14 parts, among them J1 ExpressCard, J2 Bus_M.2_Socket_M, J3 Micro_SD_Card, U1 GL823K-HCY04

Commit message: Add files via upload
Parts:
- removed C3, C4: 10uF, Capacitor_SMD:C_0603_1608Metric, symbol Device:C_Small
- removed R1, R2: 22, Resistor_SMD:R_0402_1005Metric, symbol Device:R_Small
- added F1: Fuse_Small, Fuse:Fuse_0805_2012Metric, symbol Device:Fuse_Small
- J2: footprint (none) -> Library:CONN-SMD_APCI0159-P001A
- J3: footprint Connector_Card:microSD_HC_Molex_104031-0811 -> Library:TF-SMD_TF-123-ARP9H15
Connections:
- net +3V3: now also F1.2; no longer J1.14 (3V3), J1.15 (3V3)
- net USB_D+: now also U1.15 (DP)
- net USB_D-: now also U1.16 (DM)
- net +1V5: no longer names the net of J1.10 (1V5)
- net +1V5: no longer J1.9 (1V5)
- net PCIe_RXn0 renamed PCIe_RX-
- net PCIe_RXp0 renamed PCIe_RX+
- net PCIe_TXn0 renamed PCIe_TX-
- net PCIe_TXp0 renamed PCIe_TX+
- net PEWAKE: no longer names the net of J2.54 (~{PEWAKE})
- net PEWAKE: no longer J1.11 (~{WAKE})
- net RCLKn renamed RCLK-
- net RCLKp renamed RCLK+
- new net E3V3: F1.1, J1.14 (3V3), J1.15 (3V3)
- no-connect marks 18 -> 24

Commit message: Add files via upload
Parts:
- added H1: MountingHole_Pad_MP, Library:MountingHole_3.2mm_M3_Pad_small, symbol Mechanical:MountingHole_Pad_MP
Connections:
- net GND: now also H1.MP
Changed lines of the file:
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@@
+	)
+	(symbol
+		(lib_id "power:GND")
+		(at 147.32 143.51 0)
+		(unit 1)
+		(exclude_from_sim no)
+		(in_bom yes)
+		(on_board yes)
+		(dnp no)
+		(fields_autoplaced yes)
+		(property "Reference" "#PWR06"
+			(at 147.32 149.86 0)
+			(effects
+				(font
+					(size 1.27 1.27)
+				)
+				(hide yes)
+			)
+		)
+		(property "Value" "GND"
+			(at 147.32 148.59 0)
+			(effects
+				(font
+					(size 1.27 1.27)
+				)
+				(hide yes)
+			)
+		)
+		(property "Footprint" ""
+			(at 147.32 143.51 0)
+			(effects
+				(font
+					(size 1.27 1.27)
+				)
+				(hide yes)
+			)
+		)
+		(property "Datasheet" ""
+			(at 147.32 143.51 0)
+			(effects
+				(font
+					(size 1.27 1.27)
+				)
+				(hide yes)
+			)
+		)
+		(property "Description" "Power symbol creates a global label with name \"GND\" , ground"
+			(at 147.32 143.51 0)
+			(effects
+				(font
+					(size 1.27 1.27)
+				)
+				(hide yes)
+			)
+		)
+		(pin "1"
+		)
+		(instances
+			(project "thinkmods-re"
+				(path "/7e4f06a9-8092-48d5-8507-438b9799879e"
+					(reference "#PWR06")
+					(unit 1)
+				)
+			)
+		)
 	)
 	(symbol
@@
 					(unit 1)
 				)
+			)
+		)
+	)
+	(symbol
+		(lib_id "Mechanical:MountingHole_Pad_MP")
+		(at 147.32 140.97 0)
+		(unit 1)
+		(exclude_from_sim yes)
+		(in_bom no)
+		(on_board yes)
+		(dnp no)
+		(fields_autoplaced yes)
+		(property "Reference" "H1"
+			(at 149.86 138.4299 0)
+			(effects
+				(font
+					(size 1.27 1.27)
+				)
+				(justify left)
+			)
+		)
+		(property "Value" "MountingHole_Pad_MP"
+			(at 149.86 140.9699 0)
+			(effects
+				(font
+					(size 1.27 1.27)
+				)
+				(justify left)
+			)
+		)
+		(property "Footprint" "Library:MountingHole_3.2mm_M3_Pad_small"
+			(at 147.32 140.97 0)
+			(effects
+				(font
+					(size 1.27 1.27)
+				)
+				(hide yes)
+			)
+		)
+		(property "Datasheet" "~"
+			(at 147.32 140.97 0)
+			(effects
+				(font
+					(size 1.27 1.27)
+				)
+				(hide yes)
+			)
+		)
+		(property "Description" "Mounting Hole with connection as pad named MP"
+			(at 147.32 140.97 0)
+			(effects
+				(font
+					(size 1.27 1.27)
+				)
+				(hide yes)
+			)
+		)
+		(pin "MP"
+		)
+		(instances
+			(project ""
+				(path "/7e4f06a9-8092-48d5-8507-438b9799879e"
+					(reference "H1")
+					(unit 1)
+				)
